Commit message: Depth camera added to the momodel

File: robot_model/mp_400/mp_400.urdf.xacro (robot description, xacro)
@@ -14,4 +14,6 @@
 <!-- Sick S300 - Comment/Uncomment if required  -->
 <xacro:include filename="$(find neo_mp_400)/robot_model/mp_400/xacros/sick_S300.xacro" />
+<!-- Depth camera -->
+<xacro:include filename="$(find neo_mp_400)/robot_model/mp_400/xacros/depth_camera.xacro" />
 <!-- Microscan - Comment/Uncomment if required -->
  <!-- <xacro:include filename="$(find neo_mp_400)/robot_model/mp_400/xacros/micro_scan.xacro" /> -->
@@ -122,6 +124,6 @@
   </xacro:us_sensor-->
     <!--Camera  -->
-<!-- <xacro:camera name="camera" parent="base_link">
-    <origin xyz="0 0 0.38" rpy="0 0 0" />
-  </xacro:camera> -->
+  <xacro:depth_camera name="camera" parent="base_link">
+    <origin xyz="0.158 -0.015 0.393" rpy="0 0 0" />
+  </xacro:depth_camera>
 </robot>
